Commit message: URDF change to match ROS1

File: lbr_description/urdf/iiwa14/iiwa14_description.xacro (robot description, xacro)
@@ -43,5 +43,5 @@
             </collision>
         </link>
-        <joint name="${robot_name}_A1" type="revolute">
+        <joint name="iiwa_joint_1" type="revolute">
             <origin rpy="0 0 0" xyz="0.0 0.0 0.1475" />
             <parent link="${robot_name}_link_0" />
@@ -75,5 +75,5 @@
             </collision>
         </link>
-        <joint name="${robot_name}_A2" type="revolute">
+        <joint name="iiwa_joint_2" type="revolute">
             <origin rpy="0 0 0" xyz="0.0 -0.01 0.2125" />
             <parent link="${robot_name}_link_1" />
@@ -107,5 +107,5 @@
             </collision>
         </link>
-        <joint name="${robot_name}_A3" type="revolute">
+        <joint name="iiwa_joint_3" type="revolute">
             <origin rpy="0 0 0" xyz="0.0 0.01 0.228" />
             <parent link="${robot_name}_link_2" />
@@ -139,5 +139,5 @@
             </collision>
         </link>
-        <joint name="${robot_name}_A4" type="revolute">
+        <joint name="iiwa_joint_4" type="revolute">
             <origin rpy="0 0 0" xyz="0.0 0.0105 0.192" />
             <parent link="${robot_name}_link_3" />
@@ -171,5 +171,5 @@
             </collision>
         </link>
-        <joint name="${robot_name}_A5" type="revolute">
+        <joint name="iiwa_joint_5" type="revolute">
             <origin rpy="0 0 0" xyz="0.0 -0.0105 0.2075" />
             <parent link="${robot_name}_link_4" />
@@ -203,5 +203,5 @@
             </collision>
         </link>
-        <joint name="${robot_name}_A6" type="revolute">
+        <joint name="iiwa_joint_6" type="revolute">
             <origin rpy="0 0 0" xyz="0.0 -0.0707 0.1925" />
             <parent link="${robot_name}_link_5" />
@@ -235,5 +235,5 @@
             </collision>
         </link>
-        <joint name="${robot_name}_A7" type="revolute">
+        <joint name="iiwa_joint_7" type="revolute">
             <origin rpy="0 0 0" xyz="0.0 0.0707 0.091" />
             <parent link="${robot_name}_link_6" />
